File: eagle/backpac_v3.sch (EAGLE design)
At the start: 56 parts, among them IC2 LTC3558, IC3 LT1761, IC4 LM27313, IC5 RV-2123-C2, J2 XF2-3015-1LW, Q1 12Mhz, T1 BSS84, X1 USB-MICROB

Commit message: refinements
Parts:
- added C10: 22pF, rcl:C-EUC0402
- added R16, R17: 15k, rcl:R-EU_R0402
- C18: value (none) -> 10nF; device microbuilder:CAP_CERAMIC0603MINI -> SparkFun-Capacitors:CAP0402-CAP
- C19: value (none) -> 1µF; device microbuilder:CAP_CERAMIC0603MINI -> SparkFun-Capacitors:CAP0805
Connections:
- removed net REG_EN: IC1.PIO1_7/TXD/CT32B0_MAT1
- new net ADC: C10.2, IC1.PIO1_11/AD7, R16.1, R17.1
- net +3V3: no longer T1.S
- net BAT: now also C19.1, R17.2; no longer C19.P$1
- net GND: now also C10.1, C19.2, R16.2; no longer C19.P$2
- net N$43: now also C18.1; no longer C18.P$1
- net REG_EN_: now also IC1.PIO2_6
- net VDD: now also C18.2, T1.S; no longer C18.P$2
Changed lines of the file:
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@@
 <layer number="215" name="215bmp" color="7" fill="1" visible="yes" active="yes"/>
 <layer number="216" name="216bmp" color="7" fill="1" visible="yes" active="yes"/>
+<layer number="217" name="217bmp" color="18" fill="1" visible="no" active="no"/>
+<layer number="218" name="218bmp" color="19" fill="1" visible="no" active="no"/>
+<layer number="219" name="219bmp" color="20" fill="1" visible="no" active="no"/>
+<layer number="220" name="220bmp" color="21" fill="1" visible="no" active="no"/>
+<layer number="221" name="221bmp" color="22" fill="1" visible="no" active="no"/>
+<layer number="222" name="222bmp" color="23" fill="1" visible="no" active="no"/>
+<layer number="223" name="223bmp" color="24" fill="1" visible="no" active="no"/>
+<layer number="224" name="224bmp" color="25" fill="1" visible="no" active="no"/>
 <layer number="250" name="Descript" color="3" fill="1" visible="no" active="no"/>
 <layer number="251" name="SMDround" color="12" fill="11" visible="no" active="no"/>
@@
 <part name="SUPPLY2" library="supply2" deviceset="VDD" device=""/>
 <part name="SUPPLY4" library="supply2" deviceset="VDD" device=""/>
-<part name="+3V1" library="supply1" deviceset="+3V3" device=""/>
 <part name="+3V2" library="supply1" deviceset="+3V3" device=""/>
 <part name="GND21" library="supply1" deviceset="GND" device=""/>
@@
 <part name="GND25" library="supply1" deviceset="GND" device=""/>
 <part name="C7" library="SparkFun" deviceset="CAP" device="0805" value="10µF"/>
-<part name="C18" library="microbuilder" deviceset="CAP_CERAMIC" device="0603MINI"/>
-<part name="C19" library="microbuilder" deviceset="CAP_CERAMIC" device="0603MINI"/>
+<part name="C18" library="SparkFun-Capacitors" deviceset="CAP" device="0402-CAP" value="10nF"/>
+<part name="C19" library="SparkFun-Capacitors" deviceset="CAP" device="0805" value="1µF"/>
 <part name="D1" library="diode" deviceset="DIODE-" device="DO214AC" value="B140F"/>
 <part name="L1" library="resistor" deviceset="L-EU" device="L1812" value="10µH"/>
@@
 <part name="GND30" library="supply1" deviceset="GND" device=""/>
 <part name="U$3" library="seb" deviceset="MAKE-DD_LOGO" device="'REGULAR'"/>
+<part name="SUPPLY5" library="supply2" deviceset="VDD" device=""/>
+<part name="R16" library="rcl" deviceset="R-EU_" device="R0402" value="15k"/>
+<part name="R17" library="rcl" deviceset="R-EU_" device="R0402" value="15k"/>
+<part name="GND31" library="supply1" deviceset="GND" device=""/>
+<part name="C10" library="rcl" deviceset="C-EU" device="C0402" value="22pF"/>
+<part name="GND32" library="supply1" deviceset="GND" device=""/>
 </parts>
 <sheets>
@@
 <instance part="SUPPLY2" gate="G$1" x="96.52" y="198.12" rot="R90"/>
 <instance part="SUPPLY4" gate="G$1" x="93.98" y="254" rot="R90"/>
-<instance part="+3V1" gate="G$1" x="83.82" y="246.38"/>
 <instance part="+3V2" gate="G$1" x="421.64" y="83.82"/>
 <instance part="GND21" gate="1" x="86.36" y="48.26" rot="R270"/>
@@
 <instance part="GND30" gate="1" x="106.68" y="78.74" rot="R270"/>
 <instance part="U$3" gate="G$1" x="58.42" y="289.56"/>
+<instance part="SUPPLY5" gate="G$1" x="83.82" y="246.38"/>
+<instance part="R16" gate="G$1" x="50.8" y="264.16" smashed="yes" rot="R180">
+<attribute name="NAME" x="48.768" y="262.4074" size="1.778" layer="95" rot="R180"/>
+<attribute name="VALUE" x="55.118" y="262.382" size="1.778" layer="96" rot="R180"/>
+</instance>
+<instance part="R17" gate="G$1" x="50.8" y="266.7" smashed="yes" rot="R180">
+<attribute name="NAME" x="49.022" y="270.2814" size="1.778" layer="95" rot="R180"/>
+<attribute name="VALUE" x="55.118" y="270.256" size="1.778" layer="96" rot="R180"/>
+</instance>
+<instance part="GND31" gate="1" x="43.18" y="264.16" smashed="yes" rot="R270">
+<attribute name="VALUE" x="37.084" y="263.144" size="1.778" layer="96"/>
+</instance>
+<instance part="C10" gate="G$1" x="55.88" y="259.08" smashed="yes" rot="R180">
+<attribute name="NAME" x="55.245" y="256.032" size="1.778" layer="95" rot="R90"/>
+<attribute name="VALUE" x="54.991" y="261.874" size="1.778" layer="96" rot="R90"/>
+</instance>
+<instance part="GND32" gate="1" x="55.88" y="254" smashed="yes">
+<attribute name="VALUE" x="56.896" y="247.904" size="1.778" layer="96" rot="R90"/>
+</instance>
 </instances>
 <busses>
@@
 <pinref part="IC3" gate="G$1" pin="GND"/>
 <pinref part="C7" gate="G$1" pin="1"/>
-<pinref part="C19" gate="G$1" pin="P$2"/>
+<pinref part="C19" gate="G$1" pin="2"/>
 </segment>
 <segment>
@@
 <wire x1="109.22" y1="78.74" x2="119.38" y2="78.74" width="0.1524" layer="91"/>
 </segment>
+<segment>
+<pinref part="R16" gate="G$1" pin="2"/>
+<pinref part="GND31" gate="1" pin="GND"/>
+</segment>
+<segment>
+<pinref part="C10" gate="G$1" pin="1"/>
+<pinref part="GND32" gate="1" pin="GND"/>
+</segment>
 </net>
 <net name="N$3" class="0">
@@
 <label x="88.9" y="25.4" size="1.778" layer="95"/>
 <pinref part="J2" gate="-4" pin="MS"/>
-</segment>
-<segment>
-<wire x1="83.82" y1="243.84" x2="83.82" y2="241.3" width="0.1524" layer="91"/>
-<pinref part="T1" gate="G$1" pin="S"/>
-<pinref part="+3V1" gate="G$1" pin="+3V3"/>
 </segment>
 <segment>
@@
 </segment>
 </net>
-<net name="REG_EN" class="0">
-<segment>
-<wire x1="203.2" y1="236.22" x2="210.82" y2="236.22" width="0.1524" layer="91"/>
-<label x="208.28" y="236.22" size="1.778" layer="95"/>
-<pinref part="IC1" gate="G$1" pin="PIO1_7/TXD/CT32B0_MAT1"/>
-</segment>
-</net>
 <net name="D0" class="0">
 <segment>
@@
 <pinref part="IC3" gate="G$1" pin="IN"/>
 <pinref part="IC3" gate="G$1" pin="/SHDN"/>
-<pinref part="C19" gate="G$1" pin="P$1"/>
+<pinref part="C19" gate="G$1" pin="1"/>
+</segment>
+<segment>
+<pinref part="R17" gate="G$1" pin="2"/>
+<wire x1="45.72" y1="266.7" x2="35.56" y2="266.7" width="0.1524" layer="91"/>
+<label x="35.56" y="266.7" size="1.778" layer="95"/>
 </segment>
 </net>
@@
 <pinref part="IC3" gate="G$1" pin="OUT"/>
 <pinref part="C7" gate="G$1" pin="2"/>
-<pinref part="C18" gate="G$1" pin="P$2"/>
+<pinref part="C18" gate="G$1" pin="2"/>
 <pinref part="SUPPLY1" gate="G$1" pin="VDD"/>
 </segment>
@@
 <pinref part="SUPPLY3" gate="G$1" pin="VDD"/>
 </segment>
+<segment>
+<wire x1="83.82" y1="243.84" x2="83.82" y2="241.3" width="0.1524" layer="91"/>
+<pinref part="T1" gate="G$1" pin="S"/>
+<pinref part="SUPPLY5" gate="G$1" pin="VDD"/>
+</segment>
 </net>
 <net name="N$43" class="0">
@@
 <wire x1="210.82" y1="114.3" x2="210.82" y2="116.84" width="0.1524" layer="91"/>
 <pinref part="IC3" gate="G$1" pin="BYP"/>
-<pinref part="C18" gate="G$1" pin="P$1"/>
+<pinref part="C18" gate="G$1" pin="1"/>
 </segment>
 </net>
@@
 <pinref part="R15" gate="G$1" pin="1"/>
 </segment>
+<segment>
+<pinref part="IC1" gate="G$1" pin="PIO2_6"/>
+<wire x1="203.2" y1="205.74" x2="213.36" y2="205.74" width="0.1524" layer="91"/>
+<label x="208.28" y="205.74" size="1.778" layer="95"/>
+</segment>
 </net>
 <net name="SCK" class="0">
@@
 </segment>
 </net>
+<net name="ADC" class="0">
+<segment>
+<pinref part="IC1" gate="G$1" pin="PIO1_11/AD7"/>
+<wire x1="203.2" y1="226.06" x2="210.82" y2="226.06" width="0.1524" layer="91"/>
+<label x="208.28" y="226.06" size="1.778" layer="95"/>
+</segment>
+<segment>
+<pinref part="R16" gate="G$1" pin="1"/>
+<pinref part="R17" gate="G$1" pin="1"/>
+<wire x1="55.88" y1="264.16" x2="55.88" y2="266.7" width="0.1524" layer="91"/>
+<wire x1="55.88" y1="266.7" x2="63.5" y2="266.7" width="0.1524" layer="91"/>
+<junction x="55.88" y="266.7"/>
+<label x="60.96" y="266.7" size="1.778" layer="95"/>
+<pinref part="C10" gate="G$1" pin="2"/>
+<junction x="55.88" y="264.16"/>
+</segment>
+</net>
