File: eagle/backpac_v3.brd (EAGLE design)
At the start: 37.5 x 34 mm, 56 parts, among them IC2 LTC3558, IC3 LT1761, IC4 LM27313, IC5 RV-2123-C2, J2 XF2-3015-1LW, Q1 12Mhz, T1 BSS84, X1 USB-MICROB

Commit message: refinements
Parts:
- added C10: 22pF, rcl:C0402
- added R16, R17: 15k, rcl:R0402
- C18: value (none) -> 10nF; device microbuilder:0603-MINI -> SparkFun-Capacitors:0402-CAP
- C19: value (none) -> 1µF; device microbuilder:0603-MINI -> SparkFun-Capacitors:0805
- moved U$3 30.5 mm to (1.00, 0.00), turned to 0 degrees
- moved R15 1.58 mm to (5.20, 25.2), turned to 0 degrees
- moved C5 0.45 mm to (2.20, 2.80), turned to 180 degrees
- moved C18 0.40 mm to (29.0, 3.00)
Connections:
- removed net REG_EN: IC1.47
- new net ADC: C10.2, IC1.42, R16.1, R17.1
- net +3V3: no longer T1.2
- net BAT: now also R17.2
- net GND: now also C10.1, R16.2
- net REG_EN_: now also IC1.1
- net VDD: now also T1.2
Routing:
- net ADC: track 0.00 -> 40.7 mm, vias 0 -> 2
- net VDD: track 66.3 -> 83.9 mm, vias 3 -> 5
- net REG_EN_: track 1.62 -> 10.3 mm
- net BAT: track 41.1 -> 48.9 mm
- net +3V3: track 96.6 -> 93.9 mm
- net +12V: track 70.1 -> 68.7 mm
- net GND: vias 39 -> 46

Commit message: refinement
Parts:
- moved R9 1.40 mm to (31.8, 24.9)
- moved IC5 0.40 mm to (31.2, 21.0)
Routing:
- net N$2: track 9.51 -> 10.9 mm
- net VSL: track 9.97 -> 11.4 mm
- net GND: vias 46 -> 45
Changed lines of the file:
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@@
 <attribute name="VALUE" x="30.984" y="16.303" size="0.6096" layer="27" font="vector" ratio="14"/>
 </element>
-<element name="R9" library="SparkFun" package="0805" value="50R" x="30.4" y="24.9" smashed="yes">
-<attribute name="NAME" x="32.038" y="24.5255" size="0.7" layer="25" font="vector" ratio="13"/>
-<attribute name="VALUE" x="29.484" y="24.603" size="0.6096" layer="27" font="vector" ratio="14"/>
+<element name="R9" library="SparkFun" package="0805" value="50R" x="31.8" y="24.9" smashed="yes">
+<attribute name="NAME" x="28.938" y="24.5255" size="0.7" layer="25" font="vector" ratio="13"/>
+<attribute name="VALUE" x="30.884" y="24.603" size="0.6096" layer="27" font="vector" ratio="14"/>
 </element>
 <element name="D2" library="diode" package="SOT23" value="" x="26.45" y="31.23" smashed="yes">
@@
 <attribute name="VALUE" x="8.8" y="2.9" size="0.0254" layer="27" rot="R90"/>
 </element>
-<element name="IC5" library="seb" package="RV-2123-C2" value="RV-2123-C2" x="30.8" y="21" smashed="yes" rot="R270"/>
+<element name="IC5" library="seb" package="RV-2123-C2" value="RV-2123-C2" x="31.2" y="21" smashed="yes" rot="R270"/>
 <element name="U$1" library="seb" package="B3U-3000P" value="B3U-3000P" x="15.45" y="33" smashed="yes"/>
 <element name="U$3" library="seb" package="MAKE-DD_LOGO" value="MAKE-DD_LOGO'REGULAR'" x="1" y="0"/>
@@
 <via x="16.5" y="1.4" extent="1-16" drill="0.6"/>
 <via x="31.1" y="8.7" extent="1-16" drill="0.6"/>
-<via x="32.6" y="26.3" extent="1-16" drill="0.6"/>
 <via x="23.7" y="24" extent="1-16" drill="0.6"/>
 <via x="20.2" y="25.6" extent="1-16" drill="0.6"/>
@@
 <wire x1="22.5" y1="22.8" x2="25.1" y2="22.8" width="0.254" layer="1"/>
 <wire x1="25.1" y1="22.8" x2="27.2" y2="24.9" width="0.254" layer="1"/>
-<wire x1="27.2" y1="24.9" x2="29.5" y2="24.9" width="0.254" layer="1"/>
+<wire x1="27.2" y1="24.9" x2="30.9" y2="24.9" width="0.254" layer="1"/>
 </signal>
 <signal name="VCOMH">
@@
 <contactref element="D2" pad="1"/>
 <contactref element="R9" pad="2"/>
-<wire x1="31.3" y1="26" x2="31.3" y2="24.9" width="0.254" layer="1"/>
-<wire x1="30" y1="27.3" x2="31.3" y2="26" width="0.254" layer="1"/>
-<wire x1="26.8" y1="27.3" x2="30" y2="27.3" width="0.254" layer="1"/>
-<wire x1="26.8" y1="27.3" x2="25.6" y2="28.5" width="0.254" layer="1"/>
-<wire x1="25.6" y1="28.5" x2="25.5" y2="28.6" width="0.254" layer="1"/>
+<wire x1="32.7" y1="26" x2="32.7" y2="24.9" width="0.254" layer="1"/>
+<wire x1="31.4" y1="27.3" x2="32.7" y2="26" width="0.254" layer="1"/>
+<wire x1="26.8" y1="27.3" x2="31.4" y2="27.3" width="0.254" layer="1"/>
+<wire x1="26.8" y1="27.3" x2="25.5" y2="28.6" width="0.254" layer="1"/>
 <wire x1="25.5" y1="28.6" x2="25.5" y2="30.13" width="0.254" layer="1"/>
 </signal>
@@
 <wire x1="11.6" y1="16.1" x2="11.6" y2="14.5" width="0.5" layer="1"/>
 <wire x1="11.45" y1="16.25" x2="11.6" y2="16.1" width="0.5" layer="1"/>
-<wire x1="28.1" y1="23" x2="29.25" y2="23" width="0.3048" layer="1"/>
+<wire x1="28.1" y1="23" x2="29.65" y2="23" width="0.3048" layer="1"/>
 <wire x1="29.3" y1="21.8" x2="28.1" y2="23" width="0.3048" layer="16"/>
 <wire x1="29.3" y1="6.2" x2="29.3" y2="21.8" width="0.3048" layer="16"/>
@@
 <contactref element="IC5" pad="3"/>
 <contactref element="IC1" pad="29"/>
-<wire x1="27.6" y1="21" x2="29.25" y2="21" width="0.254" layer="1"/>
+<wire x1="27.6" y1="21" x2="29.65" y2="21" width="0.254" layer="1"/>
 <wire x1="27.5" y1="20.9" x2="27.6" y2="21" width="0.254" layer="1"/>
 <wire x1="15.1" y1="17.2" x2="18" y2="17.2" width="0.254" layer="16"/>
@@
 <contactref element="IC5" pad="4"/>
 <contactref element="IC1" pad="28"/>
-<wire x1="27.6" y1="20" x2="29.25" y2="20" width="0.254" layer="1"/>
+<wire x1="27.6" y1="20" x2="29.65" y2="20" width="0.254" layer="1"/>
 <wire x1="27.2" y1="19.6" x2="27.6" y2="20" width="0.254" layer="1"/>
 <wire x1="18.7" y1="16.7" x2="18.8" y2="16.8" width="0.254" layer="1"/>
@@
 <contactref element="IC5" pad="5"/>
 <contactref element="IC1" pad="27"/>
-<wire x1="27.8" y1="19" x2="29.25" y2="19" width="0.254" layer="1"/>
+<wire x1="27.8" y1="19" x2="29.65" y2="19" width="0.254" layer="1"/>
 <wire x1="27.2" y1="18.4" x2="27.8" y2="19" width="0.254" layer="1"/>
 <wire x1="15.1" y1="16" x2="15.1" y2="15.6" width="0.254" layer="1"/>
